File: class/ARM class/Projects/simple_fan/simple_fan_schematic/simple_fan_schematic.kicad_sch (KiCad schematic)
At the start: 19 parts, among them SW1 button_stop, SW2 button_speed1, SW3 button_speed2, SW4 button_speed3, U1 NUCLEO64-F411RE, U2 PCF8574

Commit message: 🎉 'simple fan' project ppt complete
Parts:
- gave numbers to parts that had none: 1
Changed lines of the file:
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@@
   (symbol (lib_id "Motor:Fan") (at 311.15 46.99 0) (unit 1)
     (in_bom yes) (on_board yes) (dnp no) (fields_autoplaced)
-    (property "Reference" "M?" (at 316.23 45.72 0)
+    (property "Reference" "M1" (at 316.23 45.72 0)
       (effects (font (size 1.27 1.27)) (justify left))
     )
@@
       (project "simple_fan_schematic"
         (path "/f92461eb-1891-449a-a9d7-0575a2441fe9"
-          (reference "M?") (unit 1)
+          (reference "M1") (unit 1)
         )
       )
